Commit message: Added ros2_control for 6 wheels

File: description/robot_core.xacro (robot description, xacro)
@@ -56,4 +56,5 @@
         <origin xyz="${wheel_radius + wheel_separation} ${chassis_y / 2} 0" rpy="-${pi / 2} 0 0"/>
         <axis xyz="0 0 1"/>
+        <!-- <mimic joint="middle_left_wheel" multiplier="1.0"/> -->
     </joint>
     <link name="front_left_wheel">
@@ -75,6 +76,6 @@
     <gazebo reference="front_left_wheel">
         <material>Gazebo/Blue</material>
-        <mu1 value="0"/>
-        <mu2 value="0"/>
+        <!-- <mu1 value="0"/> -->
+        <!-- <mu2 value="0"/> -->
     </gazebo>
     <!-- Middle Left Wheel Link -->
@@ -110,4 +111,5 @@
         <origin xyz="-${wheel_radius + wheel_separation} ${chassis_y / 2} 0" rpy="-${pi / 2} 0 0"/>
         <axis xyz="0 0 1"/>
+        <!-- <mimic joint="middle_left_wheel" multiplier="1.0"/> -->
     </joint>
     <link name="back_left_wheel">
@@ -129,6 +131,6 @@
     <gazebo reference="back_left_wheel">
         <material>Gazebo/Blue</material>
-        <mu1 value="0"/>
-        <mu2 value="0"/>
+        <!-- <mu1 value="0"/> -->
+        <!-- <mu2 value="0"/> -->
     </gazebo>
     <!-- Front Right Wheel Link -->
@@ -138,4 +140,5 @@
         <origin xyz="${wheel_radius + wheel_separation} -${chassis_y / 2} 0" rpy="-${pi / 2} 0 ${pi}"/>
         <axis xyz="0 0 -1"/>
+        <!-- <mimic joint="middle_right_wheel" multiplier="1.0"/> -->
     </joint>
     <link name="front_right_wheel">
@@ -157,6 +160,6 @@
     <gazebo reference="front_right_wheel">
         <material>Gazebo/Blue</material>
-        <mu1 value="0"/>
-        <mu2 value="0"/>
+        <!-- <mu1 value="0"/> -->
+        <!-- <mu2 value="0"/> -->
     </gazebo>
     <!-- Middle Right Wheel Link -->
@@ -192,4 +195,5 @@
         <origin xyz="-${wheel_radius + wheel_separation} -${chassis_y / 2} 0" rpy="-${pi / 2} 0 ${pi}"/>
         <axis xyz="0 0 -1"/>
+        <!-- <mimic joint="middle_right_wheel" multiplier="1.0"/> -->
     </joint>
     <link name="back_right_wheel">
@@ -211,6 +215,6 @@
     <gazebo reference="back_right_wheel">
         <material>Gazebo/Blue</material>
-        <mu1 value="0"/>
-        <mu2 value="0"/>
+        <!-- <mu1 value="0"/> -->
+        <!-- <mu2 value="0"/> -->
     </gazebo>
 </robot>

File: description/ros2_control.xacro (robot description, xacro)
@@ -5,5 +5,35 @@
             <plugin>gazebo_ros2_control/GazeboSystem</plugin>
         </hardware>
+        <joint name="front_left_wheel_joint">
+            <!-- <param name="mimic">middle_left_wheel_joint</param>
+            <param name="multiplier">1</param> -->
+            <command_interface name="velocity">
+                <param name="min">-10</param>
+                <param name="max">10</param>
+            </command_interface>
+            <state_interface name="velocity"/>
+            <state_interface name="position"/>
+        </joint>
         <joint name="middle_left_wheel_joint">
+            <command_interface name="velocity">
+                <param name="min">-10</param>
+                <param name="max">10</param>
+            </command_interface>
+            <state_interface name="velocity"/>
+            <state_interface name="position"/>
+        </joint>
+        <joint name="back_left_wheel_joint">
+            <!-- <param name="mimic">middle_left_wheel_joint</param>
+            <param name="multiplier">1</param> -->
+            <command_interface name="velocity">
+                <param name="min">-10</param>
+                <param name="max">10</param>
+            </command_interface>
+            <state_interface name="velocity"/>
+            <state_interface name="position"/>
+        </joint>
+        <joint name="front_right_wheel_joint">
+            <!-- <param name="mimic">middle_right_wheel_joint</param>
+            <param name="multiplier">1</param> -->
             <command_interface name="velocity">
                 <param name="min">-10</param>
@@ -21,4 +51,14 @@
             <state_interface name="position"/>
         </joint>
+        <joint name="back_right_wheel_joint">
+            <!-- <param name="mimic">middle_right_wheel_joint</param>
+            <param name="multiplier">1</param> -->
+            <command_interface name="velocity">
+                <param name="min">-10</param>
+                <param name="max">10</param>
+            </command_interface>
+            <state_interface name="velocity"/>
+            <state_interface name="position"/>
+        </joint>
     </ros2_control>
 <!-- When not using Gazebo, we'll need to run ros2 run controller_manager ros2_control_node -->
